File: Hardware/Freya_SenseAndDrive_Cartridge.kicad_pcb (KiCad board)
At the start: 2 copper layers, 51.8 x 63.2 mm, 49 parts, among them J1 Screw_Terminal_01x08, J2 Grove, J3 Conn_01x02_Pin, Q1 BC847, Q10 FQD17P06TM, Q11 BC847, Q12 FQD17P06TM, Q13 BS170, Q14 BS170, Q2 FQD17P06TM, Q3 BC847, Q4 FQD17P06TM, Q5 BC847, Q6 FQD17P06TM, Q7 BC847, Q8 FQD17P06TM, Q9 BC847

Commit message: Hardware: naming in project
Parts:
- moved G*** 15.2 mm to (152.1, 89.2)
Other:
- board text added: "FREYA"
- board text added: "Rev.: 1.1"
- board text removed: "Rev.: 1.0"
