File: Hardware/Freya_SenseAndDrive_Cartridge.kicad_sch (KiCad schematic)
At the start: 40 parts, among them J1 Screw_Terminal_01x08, J2 Grove, J3 Conn_01x02_Pin, Q1 BC847, Q10 FQD17P06TM, Q11 BC847, Q12 FQD17P06TM, Q13 BS170, Q14 BS170, Q2 FQD17P06TM, Q3 BC847, Q4 FQD17P06TM, Q5 BC847, Q6 FQD17P06TM, Q7 BC847, Q8 FQD17P06TM, Q9 BC847

Commit message: Hardware: naming in project
Other:
- note added: "Copyright© 2024-2026 Sanne 'SpuQ' Santens. This design is released under the CERN OHL-W license on GitHub."
- note added: "Freya - Vivarium Control System"
- note added: "Sense'n'Drive Cartridge, Rev.: 1.1, early 2026"
- note removed: "Copyright© 2024 Sanne 'SpuQ' Santens. This design is released under the CERN OHL-W license on GitHub."
- note removed: "EDGEBERRY HARDWARE CARTRIDGE"
- note removed: "Sense'n'Drive Cartridge, Rev.: 1.0, mid 2024"
Changed lines of the file:
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@@
 		)
 	)
-	(text "Copyright© 2024 Sanne 'SpuQ' Santens. This design is released under\nthe CERN OHL-W license on GitHub."
+	(text "Copyright© 2024-2026 Sanne 'SpuQ' Santens. This design is released under\nthe CERN OHL-W license on GitHub."
 		(exclude_from_sim no)
 		(at 179.07 178.816 0)
@@
 		)
 	)
-	(text "EDGEBERRY HARDWARE CARTRIDGE"
+	(text "Freya - Vivarium Control System"
 		(exclude_from_sim no)
 		(at 178.816 172.466 0)
@@
 		)
 	)
-	(text "Sense'n'Drive Cartridge, Rev.: 1.0, mid 2024\n"
+	(text "Sense'n'Drive Cartridge, Rev.: 1.1, early 2026\n"
 		(exclude_from_sim no)
 		(at 179.07 176.53 0)
